Commit message: initial commit after fork. Gazebo works with new calibrated file. Joint names are reconfigured with new Moveit package

File: src/lerobot_description/urdf/so101.urdf.xacro (robot description, xacro)
@@ -1,5 +1,8 @@
 <?xml version="1.0"?>
-<robot name="so101" xmlns:xacro="http://www.ros.org/wiki/xacro">
-    <xacro:include filename="$(find lerobot_description)/urdf/so101_base.xacro" />
+<robot name="$(arg robot_name)" xmlns:xacro="http://www.ros.org/wiki/xacro">
+    <xacro:arg name="robot_name" default="so101" />
+    <!-- Pass through for Gazebo: use MoveIt controller config when launching with MoveIt (kienmatics_controller) -->
+    <xacro:arg name="ros2_control_config_file" default="$(find lerobot_controller)/config/so101_controllers.yaml" />
+    <xacro:include filename="$(find lerobot_description)/urdf/so101_new_calib.urdf" />
     <xacro:include filename="$(find lerobot_description)/urdf/so101_gazebo.xacro" />
     <xacro:include filename="$(find lerobot_description)/urdf/so101_ros2_control.xacro" />

File: src/lerobot_description/urdf/so101_gazebo.xacro (robot description, xacro)
@@ -1,8 +1,19 @@
 <?xml version="1.0"?>
 <robot xmlns:xacro="http://www.ros.org/wiki/xacro">
+    <!-- Expects xacro arg ros2_control_config_file (set in so101.urdf.xacro) -->
+    <!-- Fix base to world in Gazebo: root link "world" is fixed when model is spawned -->
+    <link name="world"/>
+    <joint name="world_fixed" type="fixed">
+        <parent link="world"/>
+        <child link="base_link"/>
+        <origin xyz="0 0 0" rpy="0 0 0"/>
+    </joint>
+    <gazebo reference="world">
+        <static>true</static>
+    </gazebo>
     <!-- ROS 2 Control -->
     <gazebo>
         <plugin filename="gz_ros2_control-system" name="gz_ros2_control::GazeboSimROS2ControlPlugin">
-            <parameters>$(find lerobot_controller)/config/so101_controllers.yaml</parameters>
+            <parameters>$(arg ros2_control_config_file)</parameters>
         </plugin>
     </gazebo>

File: src/lerobot_description/urdf/so101_ros2_control.xacro (robot description, xacro)
@@ -6,45 +6,51 @@
             <plugin>gz_ros2_control/GazeboSimSystem</plugin>
         </hardware>
-        <joint name="1">
+        <joint name="shoulder_pan">
             <command_interface name="position">
                 <param name="min">-1.91986</param>
                 <param name="max">1.91986</param>
             </command_interface>
-            <state_interface name="position" />
+            <state_interface name="position"/>
+            <state_interface name="velocity"/>
         </joint>
-        <joint name="2">
+        <joint name="shoulder_lift">
             <command_interface name="position">
                 <param name="min">-1.74533</param>
                 <param name="max">1.74533</param>
             </command_interface>
-            <state_interface name="position" />
+            <state_interface name="position"/>
+            <state_interface name="velocity"/>
         </joint>
-        <joint name="3">
+        <joint name="elbow_flex">
             <command_interface name="position">
                 <param name="min">-1.74533</param>
                 <param name="max">1.5708</param>
             </command_interface>
-            <state_interface name="position" />
+            <state_interface name="position"/>
+            <state_interface name="velocity"/>
         </joint>
-        <joint name="4">
+        <joint name="wrist_flex">
             <command_interface name="position">
                 <param name="min">-1.65806</param>
                 <param name="max">1.65806</param>
             </command_interface>
-            <state_interface name="position" />
+            <state_interface name="position"/>
+            <state_interface name="velocity"/>
         </joint>
-        <joint name="5">
+        <joint name="wrist_roll">
             <command_interface name="position">
                 <param name="min">-2.79253</param>
                 <param name="max">2.79253</param>
             </command_interface>
-            <state_interface name="position" />
+            <state_interface name="position"/>
+            <state_interface name="velocity"/>
         </joint>
-        <joint name="6">
+        <joint name="gripper">
             <command_interface name="position">
                 <param name="min">-0.174533</param>
                 <param name="max">1.74533</param>
             </command_interface>
-            <state_interface name="position" />
+            <state_interface name="position"/>
+            <state_interface name="velocity"/>
         </joint>
     </ros2_control>
