Commit message: Fix: error starting state is outside bounds by: [-1.82237 ] should be in the range [x -x

File: src/lerobot_description/urdf/so101_new_calib.urdf (robot description, URDF)
Before this commit: robot so101_new_calib, 8 links, 7 joints
Joints:
- joint shoulder_lift: limit lower=-1.74533 upper=1.74533 effort=10 velocity=10 -> lower=-1.82237 upper=1.74533 effort=10 velocity=10
